Commit message: fixed moments of inertia
except for wam_j7. due to it's not watertight STL, I couldn't calculate its moment of inertia. luckly, they seemed about right, except for the center of mass, which I changed to the thin shell barycenter.

File: wam_description/xacro/wam_base.urdf.xacro (robot description, xacro)
@@ -6,6 +6,6 @@
   		<inertial>
   	  		<mass value="9.97059584"/>
-	  		<origin xyz="-0.02017671 -0.26604706 -0.14071720" />
-	  		<inertia ixx="1.01232865" ixy="0.05992441" ixz="0.05388736" iyy="0.38443311" iyz="0.37488748" izz="0.82739198"/>
+	  		<origin xyz="-0.09297486 0.009962 -0.27626528" />
+	  		<inertia ixx="0.1265388512970232" ixy="-1.385690987761796e-4" ixz="0.01550612615242327e-1" iyy="0.1552999824282695" iyz="-1.970911148856444e-5" izz="0.2047880269116374"/>
 		</inertial>
 		<visual>

File: wam_description/xacro/wam_j1.urdf.xacro (robot description, xacro)
@@ -5,6 +5,6 @@
 		<inertial>
 			<mass value="10.76768767"/>
-			<origin xyz="-0.00443422 0.12189039 -0.00066489" />
-			<inertia ixx="0.29486350" ixy="-0.00795023" ixz="-0.00009311" iyy="0.11350017" iyz="0.00018711" izz="0.25065343"/>
+			<origin xyz="0 0 -0.080298" />
+			<inertia ixx="0.16930393563834" ixy="3.576235475650461e-5" ixz="6.072649354262515e-10" iyy="0.090302686185748" iyz="-8.629706291127009e-10" izz="0.14592615116211"/>
 		</inertial>
 		<visual>

File: wam_description/xacro/wam_j2.urdf.xacro (robot description, xacro)
@@ -5,6 +5,6 @@
 		<inertial>
 			<mass value="3.87493756"/>
-			<origin xyz="-0.00236983 0.03105614 0.01542114" />
-			<inertia ixx="0.02606840" ixy="-0.00001346" ixz="-0.00011701" iyy="0.01472202" iyz="0.00003659" izz="0.01934814"/>
+			<origin xyz="5.0e-6 -1.0e-6 0.050417" />
+			<inertia ixx="0.014167861011514" ixy="6.386978034996813e-6" ixz="-4.812853476190912e-7" iyy="0.016069513404066" iyz="5.368632779513262e-8" izz="0.011583377328759"/>
 		</inertial>
 		<visual>

File: wam_description/xacro/wam_j3.urdf.xacro (robot description, xacro)
@@ -5,6 +5,6 @@
 		<inertial>
 			<mass value="1.80228141"/>
-			<origin xyz="-0.03825858 0.20750770 0.00003309" />
-			<inertia ixx="0.13671601" ixy="-0.01680434" ixz="0.00000510" iyy="0.00588354" iyz="-0.00000530" izz="0.13951371"/>
+			<origin xyz="0.011841 -1.0e-6 0.44202" />
+			<inertia ixx="0.042138722542957" ixy="-2.2167540182508668e-5" ixz="-0.0022285197345" iyy="0.041776633088713" iyz="2.6306857452137573e-7" izz="0.0035131795852154"/>
 		</inertial>
 		<visual>

File: wam_description/xacro/wam_j4.urdf.xacro (robot description, xacro)
@@ -5,6 +5,6 @@
 		<inertial>
 			<mass value="1.06513649"/>
-			<origin xyz="0.01095471 -0.00002567 0.14053900" />
-			<inertia ixx="0.03952350" ixy="0.00000189" ixz="0.00003117" iyy="0.04008214" iyz="0.00000131" izz="0.00210299"/>
+			<origin xyz="-0.043013 -0.15029 -1.52e-4" />
+			<inertia ixx="6.171403900396302E-3" ixy="-3.253853817720842E-4" ixz="3.823497031140259E-7" iyy="1.1938572764041708E-3" iyz="-8.791854551099702E-6" izz="6.2223804817341365E-3"/>
 		</inertial>
 		<visual>

File: wam_description/xacro/wam_j5.urdf.xacro (robot description, xacro)
@@ -5,6 +5,6 @@
 		<inertial>
 			<mass value="0.12376019"/>
-			<origin xyz="0.00008921 0.00511217 0.00435824" />
-			<inertia ixx="0.00005587" ixy="0.00000026" ixz="0.00000000" iyy="0.00007817" iyz="-0.00000083" izz="0.00006594"/>
+			<origin xyz="0 0 -0.008768" />
+			<inertia ixx="6.084829612912498E-5" ixy="3.8639803130458314E-8" ixz="2.446427975474145E-11" iyy="9.45402767895655E-5" iyz="4.3664443852488544E-12" izz="8.662130346961971E-5"/>
 		</inertial>
 		<visual>

File: wam_description/xacro/wam_j6.urdf.xacro (robot description, xacro)
@@ -5,6 +5,6 @@
 		<inertial>
 			<mass value="0.41797364"/>
-			<origin xyz="-0.00012262 -0.01703194 0.02468336" />
-			<inertia ixx="0.00093106" ixy="0.00000148" ixz="-0.00000201" iyy="0.00049833" iyz="-0.00022162" izz="0.00057483"/>
+			<origin xyz="0.000010 -0.024192 -0.007796" />
+			<inertia ixx="6.123586601885319E-4" ixy="-2.2882704466061495E-8" ixz="7.834792016825498E-8" iyy="5.092945586817215E-4" iyz="-1.3244021879374384E-5" izz="3.0217952515151913E-4"/>
 		</inertial>
 		<visual>

File: wam_description/xacro/wam_j7.urdf.xacro (robot description, xacro)
@@ -5,5 +5,5 @@
 		<inertial>
 			<mass value="0.06864753"/>
-			<origin xyz="-0.00007974 0.00016313 -0.00323552" />
+			<origin xyz="-0.000221 0.000121 0.056434" />
 			<inertia ixx="0.00003845" ixy="-0.00000019" ixz="0.00000002" iyy="0.00003878" iyz="-0.00000004" izz="0.00007408"/>
 		</inertial>
